File: Kikad/Velocimetro/Velocimetro/Velocimetro.kicad_pcb (KiCad board)
At the start: 2 copper layers, 2 parts, among them J1 Screw_Terminal_01x03, U1 LM35-LP

Commit message: velocimetro finished
Parts:
- moved U1 1.53 mm to (164.9, 91.0), turned to 0 degrees
Connections:
- net Net-(J1-Pin_1) renamed GND
Routing:
- net GND: track 21.7 -> 0.00 mm
- net Net-(J1-Pin_2): track 20.2 -> 24.0 mm
- added copper zone on F.Cu, net GND
Changed lines of the file:
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@@
   )
   (net 0 "")
-  (net 1 "Net-(J1-Pin_1)")
+  (net 1 "GND")
   (net 2 "Net-(J1-Pin_2)")
   (net 3 "Net-(J1-Pin_3)")
@@
       (stroke (width 0.1) (type solid)) (layer "F.Fab"))
     (pad "1" thru_hole rect (at 0 0 180) (size 1.98 3.96) (drill 1.32) (layers "*.Cu" "*.Mask")
-      (net 1 "Net-(J1-Pin_1)") (pinfunction "Pin_1") (pintype "passive"))
+      (net 1 "GND") (pinfunction "Pin_1") (pintype "passive"))
     (pad "2" thru_hole oval (at 5 0 180) (size 1.98 3.96) (drill 1.32) (layers "*.Cu" "*.Mask")
       (net 2 "Net-(J1-Pin_2)") (pinfunction "Pin_2") (pintype "passive"))
@@
   )
   (footprint "Package_TO_SOT_THT:TO-92_Inline" (layer "F.Cu")
-    (at 166.382865 91.29089 180)
+    (at 164.89209 90.957727)
     (descr "TO-92 leads in-line, narrow, oval pads, drill 0.75mm (see NXP sot054_po.pdf)")
     (tags "to-92 sc-43 sc-43a sot54 PA33 transistor")
@@
     (fp_arc (start 1.27 -2.48) (mid 3.561221 -0.949055) (end 3.023625 1.753625)
       (stroke (width 0.1) (type solid)) (layer "F.Fab"))
-    (pad "1" thru_hole rect (at 0 0 180) (size 1.05 1.5) (drill 0.75) (layers "*.Cu" "*.Mask")
+    (pad "1" thru_hole rect (at 0 0) (size 1.05 1.5) (drill 0.75) (layers "*.Cu" "*.Mask")
       (net 3 "Net-(J1-Pin_3)") (pinfunction "+V_{S}") (pintype "power_in"))
-    (pad "2" thru_hole oval (at 1.27 0 180) (size 1.05 1.5) (drill 0.75) (layers "*.Cu" "*.Mask")
+    (pad "2" thru_hole oval (at 1.27 0) (size 1.05 1.5) (drill 0.75) (layers "*.Cu" "*.Mask")
       (net 2 "Net-(J1-Pin_2)") (pinfunction "V_{OUT}") (pintype "output"))
-    (pad "3" thru_hole oval (at 2.54 0 180) (size 1.05 1.5) (drill 0.75) (layers "*.Cu" "*.Mask")
-      (net 1 "Net-(J1-Pin_1)") (pinfunction "GND") (pintype "power_in"))
+    (pad "3" thru_hole oval (at 2.54 0) (size 1.05 1.5) (drill 0.75) (layers "*.Cu" "*.Mask")
+      (net 1 "GND") (pinfunction "GND") (pintype "power_in"))
     (model "${KICAD6_3DMODEL_DIR}/Package_TO_SOT_THT.3dshapes/TO-92_Inline.wrl"
       (offset (xyz 0 0 0))
@@
     )
   )
-  (gr_rect (start 157.530634 64.457661) (end 173.530634 114.457661)
+  (gr_rect (start 157.594302 64.566969) (end 173.594302 94.086969)
     (stroke (width 0.2) (type default)) (fill none) (layer "F.Cu"))
-  (segment (start 160.18 87.628025) (end 163.842865 91.29089) (width 1) (layer "F.Cu") (net 1))
-  (segment (start 160.18 71.12) (end 160.18 87.628025) (width 1) (layer "F.Cu") (net 1))
-  (segment (start 165.18 71.12) (end 165.112865 71.187135) (width 1) (layer "F.Cu") (net 2))
-  (segment (start 165.112865 71.187135) (end 165.112865 91.29089) (width 1) (layer "F.Cu") (net 2))
-  (segment (start 170.18 87.493755) (end 166.382865 91.29089) (width 1) (layer "F.Cu") (net 3))
-  (segment (start 170.18 71.12) (end 170.18 87.493755) (width 1) (layer "F.Cu") (net 3))
+  (gr_circle (center 165.991681 79.74) (end 166.991681 79.74)
+    (stroke (width 0.2) (type default)) (fill none) (layer "F.Cu"))
+  (gr_circle (center 190.5 76.2) (end 190.5 76.2)
+    (stroke (width 0.2) (type default)) (fill none) (layer "F.Cu"))
+  (segment (start 171.00309 84.366727) (end 166.16209 89.207727) (width 1) (layer "F.Cu") (net 2))
+  (segment (start 171.00309 77.02309) (end 171.00309 84.366727) (width 1) (layer "F.Cu") (net 2))
+  (segment (start 165.930092 71.950092) (end 171.00309 77.02309) (width 1) (layer "F.Cu") (net 2))
+  (segment (start 165.930092 71.036032) (end 165.930092 71.950092) (width 1) (layer "F.Cu") (net 2))
+  (segment (start 166.16209 89.207727) (end 166.16209 90.957727) (width 1) (layer "F.Cu") (net 2))
+  (segment (start 160.930092 86.995729) (end 160.930092 75.936319) (width 1) (layer "F.Cu") (net 3))
+  (segment (start 164.89209 90.957727) (end 160.930092 86.995729) (width 1) (layer "F.Cu") (net 3))
+  (segment (start 160.930092 71.036032) (end 160.930092 75.936319) (width 1) (layer "F.Cu") (net 3))
+  (zone (net 1) (net_name "GND") (layer "F.Cu") (hatch edge 0.5)
+    (connect_pads (clearance 0.5))
+    (min_thickness 0.25) (filled_areas_thickness no)
+    (fill yes (thermal_gap 0.5) (thermal_bridge_width 0.5))
+    (polygon
+      (pts
+        (xy 142.24 60.96)
+        (xy 144.78 111.76)
+        (xy 193.04 111.76)
+        (xy 190.5 55.88)
+      )
+    )
+  )
 )
