File: Kikad/Velocimetro/Velocimetro/Velocimetro.kicad_sch (KiCad schematic)
At the start: 2 parts, among them J1 Screw_Terminal_01x03, U1 LM35-LP

Commit message: velocimetro finished
Connections:
- net GND: now reaches J1.1 (Pin_1), U1.3 (GND)
Changed lines of the file:
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@@
     (stroke (width 0) (type default))
+  )
+  (global_label "GND" (shape input) (at 130.81 90.17 270) (fields_autoplaced)
+    (effects (font (size 1.27 1.27)) (justify right))
+    (property "Intersheetrefs" "${INTERSHEET_REFS}" (at 130.81 96.9463 90)
+      (effects (font (size 1.27 1.27)) (justify right) hide)
+    )
   )
   (symbol (lib_id "Sensor_Temperature:LM35-LP") (at 130.81 82.55 0) (unit 1)
@@
     )
     (pin "1")
+    (pin "2")
     (pin "3")
-    (pin "2")
     (instances
       (project "Velocimetro"
