File: Kikad/kikad_trans/kikad_trans/kikad_trans.kicad_pcb (KiCad board)
At the start: 2 copper layers, 13 parts

Commit message: cambios en kikad y en codigo completo del sender
Parts:
- moved TEMP1 3.48 mm to (123.1, 115.8), turned to 180 degrees
- moved 6.6M1 0.86 mm to (116.7, 130.6)
- moved 12M1 0.78 mm to (124.4, 134.2)
- moved CURRENT1 0.68 mm to (111.2, 125.6)
- moved 1M1 0.62 mm to (124.3, 137.9)
Connections:
- F1 pad 6: unconnected-(F1-Pin_6-Pad6) -> Net-(F1-Pin_6)
- F2 pad 16: Net-(F2-Pin_16) -> Net-(CURRENT1-Pin_2)
- F2 pad 17: Net-(CURRENT1-Pin_2) -> unconnected-(F2-Pin_17-Pad17)
- TEMP1 pad 1: 3.3V -> Net-(F1-Pin_1)
- TEMP1 pad 2: Net-(F2-Pin_16) -> Net-(F1-Pin_6)
Routing:
- net Net-(F1-Pin_6): track 0.00 -> 43.4 mm
- net Net-(F2-Pin_16): track 17.1 -> 0.00 mm
- net 3.3V: track 66.8 -> 62.6 mm
- net Net-(F1-Pin_1): track 71.4 -> 74.4 mm
- net Net-(CURRENT1-Pin_2): track 23.6 -> 25.7 mm
- net Net-(F1-Pin_7): track 55.0 -> 54.1 mm
- net Net-(F2-Pin_15): track 28.3 -> 28.8 mm

Commit message: kikad
Parts:
- moved F1 1.53 mm to (172.1, 101.5)
- moved F2 1.53 mm to (172.2, 125.5)
Routing:
- net 5V: track 47.5 -> 45.5 mm
- net Net-(CURRENT1-Pin_2): track 25.7 -> 23.9 mm
- net Net-(F1-Pin_1): track 74.4 -> 72.8 mm
- net Net-(F1-Pin_7): track 54.1 -> 52.6 mm
- net 3.3V: track 62.6 -> 61.0 mm
- net Net-(F1-Pin_6): track 43.4 -> 41.9 mm
- net Net-(Bluetooth1-Pin_5): track 11.8 -> 11.1 mm
- net Net-(Bluetooth1-Pin_4): track 11.8 -> 11.1 mm
- net Net-(F2-Pin_15): track 28.8 -> 28.2 mm
Changed lines of the file:
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@@
 	(footprint "Connector_PinSocket_2.54mm:PinSocket_1x18_P2.54mm_Vertical"
 		(layer "F.Cu")
-		(at 173.64 101.5 -90)
+		(at 172.109704 101.515795 -90)
 		(descr "Through hole straight socket strip, 1x18, 2.54mm pitch, single row (from Kicad 4.0.7), script generated")
 		(tags "Through hole socket strip THT 1x18 2.54mm single row")
@@
 	(footprint "Connector_PinSocket_2.54mm:PinSocket_1x18_P2.54mm_Vertical"
 		(layer "F.Cu")
-		(at 173.7 125.5 -90)
+		(at 172.169704 125.515795 -90)
 		(descr "Through hole straight socket strip, 1x18, 2.54mm pitch, single row (from Kicad 4.0.7), script generated")
 		(tags "Through hole socket strip THT 1x18 2.54mm single row")
@@
 	)
 	(gr_rect
-		(start 83.3 116.54)
-		(end 114.3 129.54)
-		(stroke
-			(width 0.2)
-			(type default)
-		)
-		(fill none)
-		(layer "F.Cu")
-		(net 4)
-	)
-	(gr_rect
 		(start 100 99.5)
 		(end 176 140.5)
@@
 	)
 	(segment
-		(start 154.92 131.714854)
-		(end 157.654288 128.980566)
+		(start 157.777387 128.857467)
+		(end 169.955737 128.857467)
 		(width 1)
 		(layer "F.Cu")
@@
 	)
 	(segment
-		(start 172.035027 128.980566)
-		(end 173.7 127.315593)
+		(start 154.92 131.714854)
+		(end 157.777387 128.857467)
 		(width 1)
 		(layer "F.Cu")
@@
 	)
 	(segment
-		(start 154.92 132.5)
-		(end 154.92 131.714854)
+		(start 169.955737 128.857467)
+		(end 172.169704 126.6435)
 		(width 1)
 		(layer "F.Cu")
@@
 	)
 	(segment
-		(start 157.654288 128.980566)
-		(end 172.035027 128.980566)
+		(start 154.92 132.5)
+		(end 154.92 131.714854)
 		(width 1)
 		(layer "F.Cu")
@@
 	)
 	(segment
-		(start 173.7 127.315593)
-		(end 173.7 125.5)
-		(width 1)
-		(layer "F.Cu")
-		(net 3)
-	)
-	(segment
 		(start 152.258393 137.33137)
 		(end 151.294882 138.294882)
@@
 	)
 	(segment
+		(start 172.169704 126.6435)
+		(end 172.169704 125.515795)
+		(width 1)
+		(layer "F.Cu")
+		(net 3)
+	)
+	(segment
+		(start 149.309704 125.515795)
+		(end 149.309704 127.030296)
+		(width 1)
+		(layer "F.Cu")
+		(net 5)
+	)
+	(segment
 		(start 144.12 134.5)
 		(end 144.12 132.22)
@@
 	)
 	(segment
-		(start 144.12 132.22)
-		(end 150.84 125.5)
+		(start 149.309704 127.030296)
+		(end 144.12 132.22)
 		(width 1)
 		(layer "F.Cu")
@@
 	)
 	(segment
-		(start 146.66 134.5)
-		(end 146.66 132.22)
+		(start 151.849704 127.030296)
+		(end 151.849704 125.515795)
 		(width 1)
 		(layer "F.Cu")
@@
 	(segment
 		(start 146.66 132.22)
-		(end 153.38 125.5)
+		(end 151.849704 127.030296)
+		(width 1)
+		(layer "F.Cu")
+		(net 6)
+	)
+	(segment
+		(start 146.66 134.5)
+		(end 146.66 132.22)
 		(width 1)
 		(layer "F.Cu")
@@
 	)
 	(segment
-		(start 135.6 125.006382)
-		(end 135.6 125.5)
+		(start 134.069704 125.515795)
+		(end 131.662858 123.108949)
 		(width 1)
 		(layer "F.Cu")
@@
 	)
 	(segment
-		(start 133.702567 123.108949)
-		(end 135.6 125.006382)
+		(start 131.662858 123.108949)
+		(end 129.54 123.108949)
 		(width 1)
 		(layer "F.Cu")
@@
 	(segment
 		(start 111.167658 123.108949)
-		(end 133.702567 123.108949)
+		(end 129.54 123.108949)
 		(width 1)
 		(layer "F.Cu")
@@
 	)
 	(segment
-		(start 143.891487 116.862547)
-		(end 148.800854 121.771914)
+		(start 163.345823 121.771914)
+		(end 167.089704 125.515795)
 		(width 1)
 		(layer "F.Cu")
@@
 	)
 	(segment
-		(start 128.351051 120.568949)
-		(end 132.057453 116.862547)
+		(start 111.167658 120.568949)
+		(end 128.351051 120.568949)
 		(width 1)
 		(layer "F.Cu")
@@
 	)
 	(segment
-		(start 132.057453 116.862547)
-		(end 143.891487 116.862547)
+		(start 143.891487 116.862547)
+		(end 148.800854 121.771914)
 		(width 1)
 		(layer "F.Cu")
@@
 	)
 	(segment
-		(start 111.167658 120.568949)
-		(end 128.351051 120.568949)
+		(start 132.057453 116.862547)
+		(end 143.891487 116.862547)
 		(width 1)
 		(layer "F.Cu")
@@
 	)
 	(segment
-		(start 164.891914 121.771914)
-		(end 168.62 125.5)
+		(start 148.800854 121.771914)
+		(end 163.345823 121.771914)
 		(width 1)
 		(layer "F.Cu")
@@
 	)
 	(segment
-		(start 148.800854 121.771914)
-		(end 164.891914 121.771914)
+		(start 128.351051 120.568949)
+		(end 132.057453 116.862547)
 		(width 1)
 		(layer "F.Cu")
@@
 	)
 	(segment
-		(start 106.99 103.49)
-		(end 108.692746 105.192746)
+		(start 153.192753 105.192746)
+		(end 156.869704 101.515795)
 		(width 1)
 		(layer "F.Cu")
@@
 	)
 	(segment
-		(start 108.692746 105.192746)
-		(end 154.707254 105.192746)
+		(start 106.99 103.49)
+		(end 108.692746 105.192746)
 		(width 1)
 		(layer "F.Cu")
@@
 	)
 	(segment
-		(start 154.707254 105.192746)
-		(end 158.4 101.5)
+		(start 108.692746 105.192746)
+		(end 153.192753 105.192746)
 		(width 1)
 		(layer "F.Cu")
@@
 	)
 	(segment
-		(start 155.495778 108.156588)
-		(end 160.94 102.712366)
+		(start 159.409704 102.798371)
+		(end 154.051487 108.156588)
 		(width 1)
 		(layer "F.Cu")
@@
 	)
 	(segment
-		(start 123.120831 113.285949)
-		(end 128.250192 108.156588)
+		(start 128.250192 108.156588)
+		(end 154.051487 108.156588)
 		(width 1)
 		(layer "F.Cu")
@@
 	)
 	(segment
-		(start 128.250192 108.156588)
-		(end 155.495778 108.156588)
+		(start 123.120831 113.285949)
+		(end 128.250192 108.156588)
 		(width 1)
 		(layer "F.Cu")
@@
 	)
 	(segment
-		(start 160.94 102.712366)
-		(end 160.94 101.5)
+		(start 159.409704 101.515795)
+		(end 159.409704 102.798371)
 		(width 1)
 		(layer "F.Cu")
@@
 	)
 	(segment
-		(start 127.101161 137.877879)
-		(end 138.14 126.83904)
+		(start 120.643905 134.225105)
+		(end 124.296679 137.877879)
 		(width 1)
 		(layer "F.Cu")
@@
 	)
 	(segment
-		(start 120.643905 134.225105)
-		(end 124.296679 137.877879)
+		(start 136.609704 128.369336)
+		(end 127.101161 137.877879)
 		(width 1)
 		(layer "F.Cu")
@@
 	)
 	(segment
+		(start 136.609704 125.515795)
+		(end 136.609704 128.369336)
+		(width 1)
+		(layer "F.Cu")
+		(net 18)
+	)
+	(segment
 		(start 124.296679 137.877879)
 		(end 127.101161 137.877879)
@@
 	)
 	(segment
-		(start 138.14 126.83904)
-		(end 138.14 125.5)
+		(start 130.765513 110.525954)
+		(end 163.115778 110.525954)
 		(width 1)
 		(layer "F.Cu")
-		(net 18)
+		(net 26)
 	)
 	(segment
@@
 	)
 	(segment
-		(start 164.775798 110.525954)
-		(end 173.64 101.661752)
+		(start 164.220019 109.421713)
+		(end 164.220019 109.40548)
 		(width 1)
 		(layer "F.Cu")
@@
 	)
 	(segment
-		(start 107 113.590107)
-		(end 107 113)
+		(start 163.115778 110.525954)
+		(end 164.220019 109.421713)
 		(width 1)
 		(layer "F.Cu")
@@
 	)
 	(segment
-		(start 130.765513 110.525954)
-		(end 164.775798 110.525954)
+		(start 107 113.590107)
+		(end 107 113)
 		(width 1)
 		(layer "F.Cu")
@@
 	)
 	(segment
-		(start 123.120831 115.825949)
-		(end 125.465518 115.825949)
+		(start 164.220019 109.40548)
+		(end 172.109704 101.515795)
 		(width 1)
 		(layer "F.Cu")
@@
 	)
 	(segment
-		(start 125.465518 115.825949)
-		(end 130.765513 110.525954)
+		(start 123.120831 115.825949)
+		(end 125.465518 115.825949)
 		(width 1)
 		(layer "F.Cu")
@@
 	)
 	(segment
-		(start 173.64 101.661752)
-		(end 173.64 101.5)
+		(start 109.235842 115.825949)
+		(end 107 113.590107)
 		(width 1)
 		(layer "F.Cu")
@@
 	)
 	(segment
-		(start 109.235842 115.825949)
-		(end 107 113.590107)
+		(start 125.465518 115.825949)
+		(end 130.765513 110.525954)
 		(width 1)
 		(layer "F.Cu")
@@
 		(polygon
 			(pts
-				(xy 100 99.5) (xy 100 140.5) (xy 176 140.5) (xy 176 99.5)
+				(xy 88.9 88.9) (xy 81.28 147.32) (xy 187.96 149.86) (xy 193.04 91.44)
 			)
 		)

Commit message: Kikad ahora si
Parts:
- moved 1M1 7.96 mm to (124.4, 129.9)
- moved 6.6M1 7.24 mm to (116.8, 137.9)
- moved 12M1 0.40 mm to (124.4, 133.8)
Connections:
- 6.6M1 pad 1: Net-(VOLTAJE1-Pin_1) -> Net-(VOLTAJE1-Pin_2)
- VOLTAJE1 pad 1: Net-(VOLTAJE1-Pin_1) -> GND
- VOLTAJE1 pad 2: GND -> Net-(VOLTAJE1-Pin_2)
Routing:
- net Net-(VOLTAJE1-Pin_1): track 10.5 -> 0.00 mm
- net Net-(VOLTAJE1-Pin_2): track 0.00 -> 10.00 mm
- net Net-(F2-Pin_15): track 28.2 -> 23.4 mm
Changed lines of the file:
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@@
 	(net 5 "Net-(Bluetooth1-Pin_4)")
 	(net 6 "Net-(Bluetooth1-Pin_5)")
-	(net 7 "Net-(VOLTAJE1-Pin_1)")
+	(net 7 "Net-(VOLTAJE1-Pin_2)")
 	(net 8 "Net-(CURRENT1-Pin_2)")
 	(net 9 "3.3V")
@@
 	(footprint "Resistor_THT:R_Axial_DIN0207_L6.3mm_D2.5mm_P7.62mm_Horizontal"
 		(layer "F.Cu")
-		(at 116.742495 130.638147)
+		(at 116.841219 137.877879)
 		(descr "Resistor, Axial_DIN0207 series, Axial, Horizontal, pin pitch=7.62mm, 0.25W = 1/4W, length*diameter=6.3*2.5mm^2, http://cdn-reichelt.de/documents/datenblatt/B400/1_4W%23YAG.pdf")
 		(tags "Resistor Axial_DIN0207 series Axial Horizontal pin pitch 7.62mm 0.25W = 1/4W length 6.3mm diameter 2.5mm")
@@
 			(layers "*.Cu" "*.Mask")
 			(remove_unused_layers no)
-			(net 7 "Net-(VOLTAJE1-Pin_1)")
+			(net 7 "Net-(VOLTAJE1-Pin_2)")
 			(pintype "passive")
 		)
@@
 			(layers "*.Cu" "*.Mask")
 			(remove_unused_layers no)
-			(net 7 "Net-(VOLTAJE1-Pin_1)")
+			(net 4 "GND")
 			(pinfunction "Pin_1")
 			(pintype "passive")
@@
 			(layers "*.Cu" "*.Mask")
 			(remove_unused_layers no)
-			(net 4 "GND")
+			(net 7 "Net-(VOLTAJE1-Pin_2)")
 			(pinfunction "Pin_2")
 			(pintype "passive")
@@
 	(footprint "Resistor_THT:R_Axial_DIN0207_L6.3mm_D2.5mm_P7.62mm_Horizontal"
 		(layer "F.Cu")
-		(at 124.362495 134.225105 180)
+		(at 124.428311 133.830211 180)
 		(descr "Resistor, Axial_DIN0207 series, Axial, Horizontal, pin pitch=7.62mm, 0.25W = 1/4W, length*diameter=6.3*2.5mm^2, http://cdn-reichelt.de/documents/datenblatt/B400/1_4W%23YAG.pdf")
 		(tags "Resistor Axial_DIN0207 series Axial Horizontal pin pitch 7.62mm 0.25W = 1/4W length 6.3mm diameter 2.5mm")
@@
 	(footprint "Resistor_THT:R_Axial_DIN0207_L6.3mm_D2.5mm_P7.62mm_Horizontal"
 		(layer "F.Cu")
-		(at 124.296679 137.877879 180)
+		(at 124.428311 129.914174 180)
 		(descr "Resistor, Axial_DIN0207 series, Axial, Horizontal, pin pitch=7.62mm, 0.25W = 1/4W, length*diameter=6.3*2.5mm^2, http://cdn-reichelt.de/documents/datenblatt/B400/1_4W%23YAG.pdf")
 		(tags "Resistor Axial_DIN0207 series Axial Horizontal pin pitch 7.62mm 0.25W = 1/4W length 6.3mm diameter 2.5mm")
@@
 	)
 	(segment
-		(start 114.880642 132.5)
-		(end 116.742495 130.638147)
+		(start 107 137.5)
+		(end 116.46334 137.5)
 		(width 1)
 		(layer "F.Cu")
@@
 	)
 	(segment
-		(start 107 132.5)
-		(end 114.880642 132.5)
+		(start 116.46334 137.5)
+		(end 116.841219 137.877879)
 		(width 1)
 		(layer "F.Cu")
@@
 	)
 	(segment
-		(start 124.362495 130.638147)
-		(end 124.362495 134.225105)
+		(start 124.461219 133.863119)
+		(end 124.428311 133.830211)
+		(width 1)
+		(layer "F.Cu")
+		(net 17)
+	)
+	(segment
+		(start 124.461219 137.877879)
+		(end 124.461219 133.863119)
 		(width 1)
 		(layer "F.Cu")
@@
 	)
 	(segment
-		(start 120.643905 134.225105)
-		(end 124.296679 137.877879)
+		(start 136.609704 125.740973)
+		(end 136.609704 125.515795)
 		(width 1)
 		(layer "F.Cu")
@@
 	)
 	(segment
-		(start 136.609704 128.369336)
-		(end 127.101161 137.877879)
+		(start 124.428311 129.914174)
+		(end 132.436503 129.914174)
 		(width 1)
 		(layer "F.Cu")
@@
 	)
 	(segment
-		(start 116.742495 134.225105)
-		(end 120.643905 134.225105)
+		(start 116.808311 133.830211)
+		(end 120.512274 133.830211)
 		(width 1)
 		(layer "F.Cu")
@@
 	)
 	(segment
-		(start 136.609704 125.515795)
-		(end 136.609704 128.369336)
+		(start 132.436503 129.914174)
+		(end 136.609704 125.740973)
 		(width 1)
 		(layer "F.Cu")
@@
 	)
 	(segment
-		(start 124.296679 137.877879)
-		(end 127.101161 137.877879)
+		(start 120.512274 133.830211)
+		(end 124.428311 129.914174)
 		(width 1)
 		(layer "F.Cu")
@@
 		(polygon
 			(pts
-				(xy 88.9 88.9) (xy 81.28 147.32) (xy 187.96 149.86) (xy 193.04 91.44)
+				(xy 86.400149 87.268099) (xy 78.780149 145.688099) (xy 185.460149 148.228099) (xy 190.540149 89.808099)
 			)
 		)

Commit message: ahora si lcdtm
Routing:
- net Net-(F1-Pin_6): track 41.9 -> 41.4 mm
Other:
- board text added: "Eco-Metry Transmisor"
- board text removed: "Eco-Metry Transmisor Galliano Makara Urbizu"
Changed lines of the file:
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@@
 		(layer "F.Cu")
 	)
-	(gr_text "Eco-Metry Transmisor\nGalliano\nMakara\nUrbizu"
-		(at 170.643454 120.068932 0)
-		(layer "F.Cu" knockout)
+	(gr_text "Eco-Metry Transmisor"
+		(at 174.478743 116.885095 0)
+		(layer "F.Cu")
 		(effects
 			(font
-				(size 1.3 1.3)
+				(size 1.2 1.2)
 				(thickness 0.26)
 				(bold yes)
@@
 	)
 	(segment
-		(start 159.409704 102.798371)
-		(end 154.051487 108.156588)
+		(start 128.250192 108.156588)
+		(end 123.120831 113.285949)
 		(width 1)
 		(layer "F.Cu")
@@
 	)
 	(segment
-		(start 128.250192 108.156588)
-		(end 154.051487 108.156588)
+		(start 159.409704 101.839776)
+		(end 153.092892 108.156588)
 		(width 1)
 		(layer "F.Cu")
@@
 	)
 	(segment
-		(start 123.120831 113.285949)
+		(start 153.092892 108.156588)
 		(end 128.250192 108.156588)
 		(width 1)
@@
 	(segment
 		(start 159.409704 101.515795)
-		(end 159.409704 102.798371)
+		(end 159.409704 101.839776)
 		(width 1)
 		(layer "F.Cu")
@@
 	)
 	(segment
+		(start 116.808311 133.830211)
+		(end 117.629789 133.830211)
+		(width 1)
+		(layer "F.Cu")
+		(net 18)
+	)
+	(segment
 		(start 136.609704 125.740973)
 		(end 136.609704 125.515795)
@@
 	)
 	(segment
+		(start 121.545826 129.914174)
+		(end 124.428311 129.914174)
+		(width 1)
+		(layer "F.Cu")
+		(net 18)
+	)
+	(segment
 		(start 124.428311 129.914174)
 		(end 132.436503 129.914174)
@@
 	)
 	(segment
-		(start 116.808311 133.830211)
-		(end 120.512274 133.830211)
-		(width 1)
-		(layer "F.Cu")
-		(net 18)
-	)
-	(segment
 		(start 132.436503 129.914174)
 		(end 136.609704 125.740973)
@@
 	)
 	(segment
-		(start 120.512274 133.830211)
-		(end 124.428311 129.914174)
+		(start 117.629789 133.830211)
+		(end 121.545826 129.914174)
 		(width 1)
 		(layer "F.Cu")
@@
 		(polygon
 			(pts
-				(xy 86.400149 87.268099) (xy 78.780149 145.688099) (xy 185.460149 148.228099) (xy 190.540149 89.808099)
+				(xy 90.564094 94.768614) (xy 82.944094 153.188614) (xy 303.924094 130.328614) (xy 309.004094 71.908614)
 			)
 		)
